File: hardware.kicad/controller V2/controller.kicad_pcb (KiCad board)
At the start: 2 copper layers, 74.9 x 91.4 mm, 8 parts

Commit message: update layout
Other:
- board text added: "1"
- board text added: "10"
- board text added: "11"
- board text added: "12"
- board text added: "13"
- board text added: "14"
- board text added: "15"
- board text added: "16"
- board text added: "17"
- board text added: "18"
- board text added: "19"
- board text added: "2"
- board text added: "20"
- board text added: "21"
- board text added: "22"
- board text added: "23"
- board text added: "24"
- board text added: "25"
- board text added: "26"
- board text added: "27"
- board text added: "28"
- board text added: "29"
- board text added: "3"
- board text added: "30"
- board text added: "31"
- board text added: "32"
- board text added: "4"
- board text added: "5"
- board text added: "6"
- board text added: "7"
- board text added: "8"
- board text added: "9"
- board text added: "Channel 1-16"
- board text added: "Channel 17-32"
- board text added: "Channel Controller"
- board text removed: "Channel V2"
Changed lines of the file:
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@@
   (general
     (thickness 1.6)
-    (drawings 115)
+    (drawings 156)
     (tracks 287)
     (zones 0)
@@
   (layers
     (0 F.Cu signal)
-    (31 B.Cu signal hide)
-    (32 B.Adhes user hide)
-    (33 F.Adhes user hide)
-    (34 B.Paste user hide)
+    (31 B.Cu signal)
+    (32 B.Adhes user)
+    (33 F.Adhes user)
+    (34 B.Paste user)
     (35 F.Paste user)
-    (36 B.SilkS user hide)
+    (36 B.SilkS user)
     (37 F.SilkS user)
-    (38 B.Mask user hide)
+    (38 B.Mask user)
     (39 F.Mask user)
-    (40 Dwgs.User user hide)
-    (41 Cmts.User user hide)
-    (42 Eco1.User user hide)
-    (43 Eco2.User user hide)
+    (40 Dwgs.User user)
+    (41 Cmts.User user)
+    (42 Eco1.User user)
+    (43 Eco2.User user)
     (44 Edge.Cuts user)
-    (45 Margin user hide)
-    (46 B.CrtYd user hide)
+    (45 Margin user)
+    (46 B.CrtYd user)
     (47 F.CrtYd user)
-    (48 B.Fab user hide)
+    (48 B.Fab user)
     (49 F.Fab user)
   )
@@
     (solder_mask_min_width 0.25)
     (aux_axis_origin 0 0)
-    (visible_elements FFFFFF7F)
+    (visible_elements 7FFFF7FF)
     (pcbplotparams
       (layerselection 0x010fc_ffffffff)
@@
     (descr "Through hole angled pin header, 2x10, 2.54mm pitch, 6mm pin length, double rows")
     (tags "Through hole angled pin header THT 2x10 2.54mm double row")
-    (fp_text reference REF** (at 5.655 -2.27) (layer F.SilkS) hide
-      (effects (font (size 1 1) (thickness 0.15)))
-    )
-    (fp_text value 2x10_P2.54mm_Horizontal (at 13.97 11.43 -90) (layer F.Fab) hide
+    (fp_text reference REF** (at 0 0) (layer F.SilkS) hide
+      (effects (font (size 1 1) (thickness 0.15)))
+    )
+    (fp_text value 2x10_P2.54mm_Horizontal (at 5.08 10.16 -90) (layer F.Fab) hide
       (effects (font (size 1 1) (thickness 0.15)))
     )
@@
     (descr "Through hole angled pin header, 2x10, 2.54mm pitch, 6mm pin length, double rows")
     (tags "Through hole angled pin header THT 2x10 2.54mm double row")
-    (fp_text reference REF** (at 5.655 -2.27) (layer F.SilkS) hide
+    (fp_text reference REF** (at 1.27 0) (layer F.SilkS) hide
       (effects (font (size 1 1) (thickness 0.15)))
     )
@@
     )
   )
-  (gr_text "Channel V2" (at 110.49 64.77 270) (layer F.SilkS)
+  (gr_text "Channel 17-32" (at 161.29 92.71) (layer F.SilkS)
+    (effects (font (size 1 1) (thickness 0.2)))
+  )
+  (gr_text "Channel 1-16" (at 161.29 49.53) (layer F.SilkS)
+    (effects (font (size 1 1) (thickness 0.2)))
+  )
+  (gr_text 20 (at 162.56 114.3) (layer F.SilkS)
+    (effects (font (size 0.8 0.8) (thickness 0.15)) (justify left))
+  )
+  (gr_text 23 (at 166.37 109.22) (layer F.SilkS)
+    (effects (font (size 0.8 0.8) (thickness 0.15)) (justify left))
+  )
+  (gr_text 25 (at 166.37 106.68) (layer F.SilkS)
+    (effects (font (size 0.8 0.8) (thickness 0.15)) (justify left))
+  )
+  (gr_text 17 (at 166.37 116.84) (layer F.SilkS)
+    (effects (font (size 0.8 0.8) (thickness 0.15)) (justify left))
+  )
+  (gr_text 18 (at 162.56 116.84) (layer F.SilkS)
+    (effects (font (size 0.8 0.8) (thickness 0.15)) (justify left))
+  )
+  (gr_text 21 (at 166.37 111.76) (layer F.SilkS)
+    (effects (font (size 0.8 0.8) (thickness 0.15)) (justify left))
+  )
+  (gr_text Vcc (at 162.56 120.65) (layer F.SilkS)
+    (effects (font (size 0.8 0.8) (thickness 0.15)) (justify left))
+  )
+  (gr_text 26 (at 162.56 106.68) (layer F.SilkS)
+    (effects (font (size 0.8 0.8) (thickness 0.15)) (justify left))
+  )
+  (gr_text 19 (at 166.37 114.3) (layer F.SilkS)
+    (effects (font (size 0.8 0.8) (thickness 0.15)) (justify left))
+  )
+  (gr_text 22 (at 162.56 111.76) (layer F.SilkS)
+    (effects (font (size 0.8 0.8) (thickness 0.15)) (justify left))
+  )
+  (gr_text 27 (at 166.37 104.14) (layer F.SilkS)
+    (effects (font (size 0.8 0.8) (thickness 0.15)) (justify left))
+  )
+  (gr_text 28 (at 162.56 104.14) (layer F.SilkS)
+    (effects (font (size 0.8 0.8) (thickness 0.15)) (justify left))
+  )
+  (gr_text 30 (at 162.56 101.6) (layer F.SilkS)
+    (effects (font (size 0.8 0.8) (thickness 0.15)) (justify left))
+  )
+  (gr_text 29 (at 166.37 101.6) (layer F.SilkS)
+    (effects (font (size 0.8 0.8) (thickness 0.15)) (justify left))
+  )
+  (gr_text GND (at 166.37 95.25) (layer F.SilkS)
+    (effects (font (size 0.8 0.8) (thickness 0.15)) (justify left))
+  )
+  (gr_text 32 (at 162.56 99.06) (layer F.SilkS)
+    (effects (font (size 0.8 0.8) (thickness 0.15)) (justify left))
+  )
+  (gr_text Vcc (at 166.37 120.65) (layer F.SilkS)
+    (effects (font (size 0.8 0.8) (thickness 0.15)) (justify left))
+  )
+  (gr_text GND (at 162.56 95.25) (layer F.SilkS)
+    (effects (font (size 0.8 0.8) (thickness 0.15)) (justify left))
+  )
+  (gr_text 31 (at 166.37 99.06) (layer F.SilkS)
+    (effects (font (size 0.8 0.8) (thickness 0.15)) (justify left))
+  )
+  (gr_text 24 (at 162.56 109.22) (layer F.SilkS)
+    (effects (font (size 0.8 0.8) (thickness 0.15)) (justify left))
+  )
+  (gr_text GND (at 162.56 52.07) (layer F.SilkS)
+    (effects (font (size 0.8 0.8) (thickness 0.15)) (justify left))
+  )
+  (gr_text GND (at 166.37 52.07) (layer F.SilkS)
+    (effects (font (size 0.8 0.8) (thickness 0.15)) (justify left))
+  )
+  (gr_text Vcc (at 166.37 77.47) (layer F.SilkS)
+    (effects (font (size 0.8 0.8) (thickness 0.15)) (justify left))
+  )
+  (gr_text 16 (at 162.56 55.88) (layer F.SilkS)
+    (effects (font (size 0.8 0.8) (thickness 0.15)) (justify left))
+  )
+  (gr_text 15 (at 166.37 55.88) (layer F.SilkS)
+    (effects (font (size 0.8 0.8) (thickness 0.15)) (justify left))
+  )
+  (gr_text "13\n" (at 166.37 58.42) (layer F.SilkS)
+    (effects (font (size 0.8 0.8) (thickness 0.15)) (justify left))
+  )
+  (gr_text 14 (at 162.56 58.42) (layer F.SilkS)
+    (effects (font (size 0.8 0.8) (thickness 0.15)) (justify left))
+  )
+  (gr_text 12 (at 162.56 60.96) (layer F.SilkS)
+    (effects (font (size 0.8 0.8) (thickness 0.15)) (justify left))
+  )
+  (gr_text 11 (at 166.37 60.96) (layer F.SilkS)
+    (effects (font (size 0.8 0.8) (thickness 0.15)) (justify left))
+  )
+  (gr_text 6 (at 162.56 68.58) (layer F.SilkS)
+    (effects (font (size 0.8 0.8) (thickness 0.15)) (justify left))
+  )
+  (gr_text 8 (at 162.56 66.04) (layer F.SilkS)
+    (effects (font (size 0.8 0.8) (thickness 0.15)) (justify left))
+  )
+  (gr_text 10 (at 162.56 63.5) (layer F.SilkS)
+    (effects (font (size 0.8 0.8) (thickness 0.15)) (justify left))
+  )
+  (gr_text 9 (at 166.37 63.5) (layer F.SilkS)
+    (effects (font (size 0.8 0.8) (thickness 0.15)) (justify left))
+  )
+  (gr_text 7 (at 166.37 66.04) (layer F.SilkS)
+    (effects (font (size 0.8 0.8) (thickness 0.15)) (justify left))
+  )
+  (gr_text 5 (at 166.37 68.58) (layer F.SilkS)
+    (effects (font (size 0.8 0.8) (thickness 0.15)) (justify left))
+  )
+  (gr_text 4 (at 162.56 71.12) (layer F.SilkS)
+    (effects (font (size 0.8 0.8) (thickness 0.15)) (justify left))
+  )
+  (gr_text 3 (at 166.37 71.12) (layer F.SilkS)
+    (effects (font (size 0.8 0.8) (thickness 0.15)) (justify left))
+  )
+  (gr_text 2 (at 162.56 73.66) (layer F.SilkS)
+    (effects (font (size 0.8 0.8) (thickness 0.15)) (justify left))
+  )
+  (gr_text 1 (at 166.37 73.66) (layer F.SilkS)
+    (effects (font (size 0.8 0.8) (thickness 0.15)) (justify left))
+  )
+  (gr_text Vcc (at 162.56 77.47) (layer F.SilkS)
+    (effects (font (size 0.8 0.8) (thickness 0.15)) (justify left))
+  )
+  (gr_text "Channel Controller" (at 110.49 64.77 270) (layer F.SilkS)
     (effects (font (size 1 1) (thickness 0.2)))
   )
@@
   (gr_poly (pts (xy 120.65 59.69) (xy 120.65 58.42) (xy 121.92 58.42) (xy 121.92 59.69)) (layer F.SilkS) (width 0.1))
   (gr_poly (pts (xy 119.38 58.42) (xy 119.38 57.15) (xy 120.65 57.15) (xy 120.65 58.42)) (layer F.SilkS) (width 0.1))
-  (dimension 64.77 (width 0.1) (layer Dwgs.User)
-    (gr_text "64.770 mm" (at 136.525 146.08) (layer Dwgs.User)
-      (effects (font (size 1 1) (thickness 0.1)))
-    )
-    (feature1 (pts (xy 104.14 142.24) (xy 104.14 145.366421)))
-    (feature2 (pts (xy 168.91 142.24) (xy 168.91 145.366421)))
-    (crossbar (pts (xy 168.91 144.78) (xy 104.14 144.78)))
-    (arrow1a (pts (xy 104.14 144.78) (xy 105.266504 144.193579)))
-    (arrow1b (pts (xy 104.14 144.78) (xy 105.266504 145.366421)))
-    (arrow2a (pts (xy 168.91 144.78) (xy 167.783496 144.193579)))
-    (arrow2b (pts (xy 168.91 144.78) (xy 167.783496 145.366421)))
-  )
   (dimension 91.44 (width 0.12) (layer F.SilkS)
     (gr_text "91.440 mm" (at 181.56 86.36 270) (layer F.SilkS)

Commit message: no message
Parts:
- added  : , Connector_PinHeader_2.54mm:PinHeader_1x06_P2.54mm_Vertical, F.Cu at (121.9, 73.7)
- added  : , Connector_PinHeader_2.54mm:PinHeader_1x06_P2.54mm_Vertical, F.Cu at (127.0, 73.7)
Routing:
- net (no net): track 1381.6 -> 1412.1 mm
Other:
- board size 74.9 x 91.4 mm -> 78.7 x 91.4 mm
- rule trace_min: 0.2 -> 0.254
- rule via_min_size: 0.4 -> 0.2
- board text removed: "Channel Controller"
- board text removed: "github.com/s910324/Relay-Controller"

Commit message: update ground pin layout
Routing:
- net (no net): track 1412.1 -> 1408.3 mm
Changed lines of the file:
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@@
   (segment (start 151.13 49.53) (end 146.05 49.53) (width 0.254) (layer B.Cu) (net 0))
   (segment (start 146.05 83.82) (end 152.4 83.82) (width 0.254) (layer F.Cu) (net 0))
-  (via (at 135.89 90.17) (size 0.8) (drill 0.4) (layers F.Cu B.Cu) (net 0))
   (via (at 133.35 97.79) (size 0.8) (drill 0.4) (layers F.Cu B.Cu) (net 0))
   (via (at 130.81 92.71) (size 0.8) (drill 0.4) (layers F.Cu B.Cu) (net 0))
@@
   (segment (start 151.13 92.71) (end 146.05 92.71) (width 0.254) (layer B.Cu) (net 0))
   (segment (start 138.43 105.41) (end 135.89 105.41) (width 0.254) (layer B.Cu) (net 0))
-  (segment (start 135.89 90.17) (end 135.89 90.17) (width 0.254) (layer B.Cu) (net 0))
   (segment (start 132.08 95.25) (end 132.08 95.25) (width 0.254) (layer B.Cu) (net 0))
   (segment (start 134.62 87.63) (end 134.62 83.82) (width 0.254) (layer F.Cu) (net 0))
@@
   (segment (start 135.89 93.98) (end 135.89 93.98) (width 0.254) (layer B.Cu) (net 0))
   (via (at 135.89 93.98) (size 0.8) (drill 0.4) (layers F.Cu B.Cu) (net 0))
-  (segment (start 135.89 90.17) (end 127 90.17) (width 0.254) (layer B.Cu) (net 0))
-  (segment (start 127 90.17) (end 127 88.9) (width 0.254) (layer B.Cu) (net 0))
   (segment (start 107.95 104.14) (end 109.22 102.87) (width 0.254) (layer B.Cu) (net 0))
   (segment (start 132.08 102.87) (end 132.08 102.87) (width 0.254) (layer B.Cu) (net 0))
@@
   (segment (start 121.92 71.12) (end 127 71.12) (width 0.254) (layer B.Cu) (net 0))
   (segment (start 127 73.66) (end 121.92 73.66) (width 0.254) (layer B.Cu) (net 0))
+  (segment (start 135.89 90.17) (end 135.89 90.17) (width 0.254) (layer B.Cu) (net 0))
+  (via (at 135.89 90.17) (size 0.8) (drill 0.4) (layers F.Cu B.Cu) (net 0))
+  (segment (start 133.27 88.98) (end 133.35 88.9) (width 0.254) (layer B.Cu) (net 0))
+  (segment (start 127 88.98) (end 133.27 88.98) (width 0.254) (layer B.Cu) (net 0))
 )
